File: kicad/Relay control/optocupler.sch (KiCad schematic (older format))
At the start: 63 parts, among them J1 Conn_01x10_Female, J2 Conn_01x04_Female, J3 Conn_01x03_Female, J4 Conn_01x04_Male, J5 Conn_01x04_Male, J6 Conn_01x04_Male, J7 Conn_01x04_Male, J8 Conn_01x04_Female, J9 Conn_01x03_Female, Q1 BS170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

Commit message: rst pin for nano
Parts:
- removed J2: Conn_01x04_Female, Connector_PinSocket_2.54mm:PinSocket_1x04_P2.54mm_Vertical, symbol Connector:Conn_01x04_Female
- added J2: Conn_01x05_Female, Connector_PinSocket_2.54mm:PinSocket_1x05_P2.54mm_Vertical, symbol Connector:Conn_01x05_Female
- J4, J5, J6, J7: footprint Connector_JST:JST_NV_B04P-NV_1x04_P5.00mm_Vertical -> Connector_Phoenix_MSTB:PhoenixContact_MSTBVA_2,5_4-G_1x04_P5.00mm_Vertical
Connections:
- net at A1.1 (D1/TX): now also J2.1 (Pin_1)
- net at A1.2 (D0/RX): now also J2.2 (Pin_2)
- net at A1.29 (GND), A1.4 (GND), C11.2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: now also J2.4 (Pin_4)
- net at A1.3 (RESET): now also J2.5 (Pin_5)
- net at A1.30 (VIN), C9.2: now also J2.3 (Pin_3)
- no-connect marks 4 -> 3
Changed lines of the file:
@@
 F 0 "J4" H 6873 1330 50  0000 R CNN
 F 1 "Conn_01x04_Male" H 6873 1421 50  0000 R CNN
-F 2 "Connector_JST:JST_NV_B04P-NV_1x04_P5.00mm_Vertical" H 6900 1450 50  0001 C CNN
+F 2 "Connector_Phoenix_MSTB:PhoenixContact_MSTBVA_2,5_4-G_1x04_P5.00mm_Vertical" H 6900 1450 50  0001 C CNN
 F 3 "~" H 6900 1450 50  0001 C CNN
 	1    6900 1450
@@
 F 0 "J5" H 6873 2430 50  0000 R CNN
 F 1 "Conn_01x04_Male" H 6873 2521 50  0000 R CNN
-F 2 "Connector_JST:JST_NV_B04P-NV_1x04_P5.00mm_Vertical" H 6900 2550 50  0001 C CNN
+F 2 "Connector_Phoenix_MSTB:PhoenixContact_MSTBVA_2,5_4-G_1x04_P5.00mm_Vertical" H 6900 2550 50  0001 C CNN
 F 3 "~" H 6900 2550 50  0001 C CNN
 	1    6900 2550
@@
 F 0 "J6" H 6873 3530 50  0000 R CNN
 F 1 "Conn_01x04_Male" H 6873 3621 50  0000 R CNN
-F 2 "Connector_JST:JST_NV_B04P-NV_1x04_P5.00mm_Vertical" H 6900 3650 50  0001 C CNN
+F 2 "Connector_Phoenix_MSTB:PhoenixContact_MSTBVA_2,5_4-G_1x04_P5.00mm_Vertical" H 6900 3650 50  0001 C CNN
 F 3 "~" H 6900 3650 50  0001 C CNN
 	1    6900 3650
@@
 F 0 "J7" H 6873 4630 50  0000 R CNN
 F 1 "Conn_01x04_Male" H 6873 4721 50  0000 R CNN
-F 2 "Connector_JST:JST_NV_B04P-NV_1x04_P5.00mm_Vertical" H 6900 4750 50  0001 C CNN
+F 2 "Connector_Phoenix_MSTB:PhoenixContact_MSTBVA_2,5_4-G_1x04_P5.00mm_Vertical" H 6900 4750 50  0001 C CNN
 F 3 "~" H 6900 4750 50  0001 C CNN
 	1    6900 4750
@@
 	5800 5700 5800 6200
 NoConn ~ 3050 2700
-NoConn ~ 3050 2400
 NoConn ~ 3050 2300
 NoConn ~ 2650 1900
@@
 Wire Wire Line
 	3250 1400 3250 4000
-$Comp
-L Connector:Conn_01x04_Female J2
-U 1 1 5C8A5D08
-P 2050 1050
-F 0 "J2" V 1990 762 50  0000 R CNN
-F 1 "Conn_01x04_Female" V 1899 762 50  0000 R CNN
-F 2 "Connector_PinSocket_2.54mm:PinSocket_1x04_P2.54mm_Vertical" H 2050 1050 50  0001 C CNN
-F 3 "~" H 2050 1050 50  0001 C CNN
-	1    2050 1050
-	0    -1   -1   0
-$EndComp
 $Comp
 L Device:C C9
@@
 Wire Wire Line
 	4800 1800 4850 1800
+$Comp
+L Connector:Conn_01x05_Female J2
+U 1 1 5C72CC15
+P 2150 1050
+F 0 "J2" V 2090 762 50  0000 R CNN
+F 1 "Conn_01x05_Female" V 1999 762 50  0000 R CNN
+F 2 "Connector_PinSocket_2.54mm:PinSocket_1x05_P2.54mm_Vertical" H 2150 1050 50  0001 C CNN
+F 3 "~" H 2150 1050 50  0001 C CNN
+	1    2150 1050
+	0    -1   -1   0
+$EndComp
+Wire Wire Line
+	3050 2400 3150 2400
+Wire Wire Line
+	3150 2400 3150 1600
+Wire Wire Line
+	3150 1600 2350 1600
+Wire Wire Line
+	2350 1600 2350 1250
 $EndSCHEMATC
