File: kicad/Relay control/optocupler.kicad_pcb (KiCad board)
At the start: 2 copper layers, 100 x 100 mm, 63 parts, among them J1 Conn_01x10_Female, J2 Conn_01x04_Female, J3 Conn_01x03_Female, J4 Conn_01x04_Male, J5 Conn_01x04_Male, J6 Conn_01x04_Male, J7 Conn_01x04_Male, J8 Conn_01x04_Female, J9 Conn_01x03_Female, Q1 BS170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

Commit message: rst pin for nano
Parts:
- J2: value Conn_01x04_Female -> Conn_01x05_Female; footprint Connector_PinSocket_2.54mm:PinSocket_1x04_P2.54mm_Vertical -> Connector_PinSocket_2.54mm:PinSocket_1x05_P2.54mm_Vertical
- J4, J5, J6, J7: footprint Connector_JST:JST_NV_B04P-NV_1x04_P5.00mm_Vertical -> Connector_Phoenix_MSTB:PhoenixContact_MSTBVA_2,5_4-G_1x04_P5.00mm_Vertical
Routing:
- net Net-(A1-Pad3): track 0.00 -> 27.9 mm

Commit message: update pcb
Routing:
- net (no net): vias 0 -> 6
Other:
- outline, holes or cut-outs redrawn
Changed lines of the file:
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@@
   (general
     (thickness 1.6)
-    (drawings 23)
-    (tracks 320)
+    (drawings 17)
+    (tracks 326)
     (zones 0)
     (modules 63)
@@
     (effects (font (size 1.5 1.5) (thickness 0.3)))
   )
-  (gr_circle (center 92.5 105) (end 92.5 103.5) (layer Edge.Cuts) (width 0.15))
-  (gr_circle (center 187.5 105) (end 187.5 103.5) (layer Edge.Cuts) (width 0.15))
-  (gr_circle (center 92.5 152.5) (end 92.5 151) (layer Edge.Cuts) (width 0.15))
-  (gr_circle (center 187.5 152.5) (end 187.5 151) (layer Edge.Cuts) (width 0.15))
-  (gr_circle (center 187.5 57.5) (end 187.5 56) (layer Edge.Cuts) (width 0.15))
-  (gr_circle (center 92.5 57.5) (end 92.5 56) (layer Edge.Cuts) (width 0.15))
   (gr_line (start 190 55) (end 90 55) (layer Edge.Cuts) (width 0.15))
   (gr_line (start 190 155) (end 190 55) (layer Edge.Cuts) (width 0.15))
   (gr_line (start 90 155) (end 190 155) (layer Edge.Cuts) (width 0.15))
   (gr_line (start 90 55) (end 90 155) (layer Edge.Cuts) (width 0.15))
+  (via (at 187.5 105) (size 3.1) (drill 3) (layers F.Cu B.Cu) (net 0))
+  (via (at 187.5 57.5) (size 3.1) (drill 3) (layers F.Cu B.Cu) (net 0))
+  (via (at 187.5 152.5) (size 3.1) (drill 3) (layers F.Cu B.Cu) (net 0))
+  (via (at 92.5 152.5) (size 3.1) (drill 3) (layers F.Cu B.Cu) (net 0))
+  (via (at 92.5 105) (size 3.1) (drill 3) (layers F.Cu B.Cu) (net 0))
+  (via (at 92.5 57.5) (size 3.1) (drill 3) (layers F.Cu B.Cu) (net 0))
   (segment (start 101.75 58) (end 103 58) (width 0.4) (layer F.Cu) (net 1))
   (segment (start 99 60.75) (end 101.75 58) (width 0.4) (layer F.Cu) (net 1))
