File: kicad/Display/display.kicad_pcb (KiCad board)
At the start: 2 copper layers, 100 x 100 mm, 36 parts, among them IC1 RaspberryPiZeroW, J1 Conn_01x02_Female, J2 Conn_01x05_Female, SW1 SW_Push_Dual, SW2 SW_Push_Dual, SW3 SW_Push_Dual, SW4 SW_Push_Dual, U1 LM7805_TO220

Commit message: update pcb
Parts:
- removed TFT1: SPI_TFT, display:SPI_TFT
- added REF**: pad, display:pad, F.Cu at (132.1, 137.2)
- added REF**: pad, display:pad, F.Cu at (134.6, 134.6)
- added REF**: pad, display:pad, F.Cu at (149.9, 127.0)
- added REF**: pad, display:pad, F.Cu at (147.3, 127.0)
- added REF**: pad, display:pad, F.Cu at (149.9, 124.5)
- added REF**: pad, display:pad, F.Cu at (147.3, 114.3)
- added REF**: pad, display:pad, F.Cu at (149.9, 119.4)
- added REF**: pad, display:pad, F.Cu at (152.4, 114.3)
- added REF**: pad, display:pad, F.Cu at (154.9, 111.8)
- added REF**: pad, display:pad, F.Cu at (147.3, 111.8)
- added REF**: pad, display:pad, F.Cu at (147.3, 119.4)
- added REF**: pad, display:pad, F.Cu at (152.4, 116.8)
- added REF**: pad, display:pad, F.Cu at (132.1, 134.6)
- added REF**: pad, display:pad, F.Cu at (154.9, 114.3)
- added REF**: pad, display:pad, F.Cu at (152.4, 111.8)
- added REF**: pad, display:pad, F.Cu at (149.9, 111.8)
- added REF**: pad, display:pad, F.Cu at (152.4, 119.4)
- added REF**: pad, display:pad, F.Cu at (149.9, 116.8)
- added REF**: pad, display:pad, F.Cu at (147.3, 116.8)
- added REF**: pad, display:pad, F.Cu at (149.9, 114.3)
- added REF**: pad, display:pad, F.Cu at (129.5, 119.4)
- added REF**: pad, display:pad, F.Cu at (134.6, 119.4)
- added REF**: pad, display:pad, F.Cu at (132.1, 116.8)
- added REF**: pad, display:pad, F.Cu at (165.1, 137.2)
- added REF**: pad, display:pad, F.Cu at (134.6, 114.3)
- added REF**: pad, display:pad, F.Cu at (132.1, 119.4)
- added REF**: pad, display:pad, F.Cu at (134.6, 116.8)
- added REF**: pad, display:pad, F.Cu at (127.0, 124.5)
- added REF**: pad, display:pad, F.Cu at (129.5, 129.5)
- added REF**: pad, display:pad, F.Cu at (132.1, 124.5)
- added REF**: pad, display:pad, F.Cu at (134.6, 121.9)
- added REF**: pad, display:pad, F.Cu at (127.0, 121.9)
- added REF**: pad, display:pad, F.Cu at (127.0, 129.5)
- added REF**: pad, display:pad, F.Cu at (134.6, 129.5)
- added REF**: pad, display:pad, F.Cu at (162.6, 137.2)
- added REF**: pad, display:pad, F.Cu at (132.1, 127.0)
- added REF**: pad, display:pad, F.Cu at (134.6, 124.5)
- added REF**: pad, display:pad, F.Cu at (132.1, 121.9)
- added REF**: pad, display:pad, F.Cu at (129.5, 121.9)
- added REF**: pad, display:pad, F.Cu at (132.1, 129.5)
- added REF**: pad, display:pad, F.Cu at (129.5, 127.0)
- added REF**: pad, display:pad, F.Cu at (127.0, 127.0)
- added REF**: pad, display:pad, F.Cu at (134.6, 127.0)
- added REF**: pad, display:pad, F.Cu at (129.5, 124.5)
- added REF**: pad, display:pad, F.Cu at (137.2, 124.5)
- added REF**: pad, display:pad, F.Cu at (160.0, 137.2)
- added REF**: pad, display:pad, F.Cu at (139.7, 129.5)
- added REF**: pad, display:pad, F.Cu at (142.2, 124.5)
- added REF**: pad, display:pad, F.Cu at (144.8, 121.9)
- added REF**: pad, display:pad, F.Cu at (137.2, 121.9)
- added REF**: pad, display:pad, F.Cu at (137.2, 129.5)
- added REF**: pad, display:pad, F.Cu at (144.8, 129.5)
- added REF**: pad, display:pad, F.Cu at (142.2, 127.0)
- added REF**: pad, display:pad, F.Cu at (144.8, 124.5)
- added REF**: pad, display:pad, F.Cu at (142.2, 121.9)
- added REF**: pad, display:pad, F.Cu at (139.7, 121.9)
- added REF**: pad, display:pad, F.Cu at (157.5, 137.2)
- added REF**: pad, display:pad, F.Cu at (142.2, 129.5)
- added REF**: pad, display:pad, F.Cu at (139.7, 127.0)
- added REF**: pad, display:pad, F.Cu at (137.2, 127.0)
- added REF**: pad, display:pad, F.Cu at (144.8, 127.0)
- added REF**: pad, display:pad, F.Cu at (139.7, 124.5)
- added REF**: pad, display:pad, F.Cu at (137.2, 114.3)
- added REF**: pad, display:pad, F.Cu at (139.7, 119.4)
- added REF**: pad, display:pad, F.Cu at (142.2, 114.3)
- added REF**: pad, display:pad, F.Cu at (144.8, 111.8)
- added REF**: pad, display:pad, F.Cu at (137.2, 111.8)
- added REF**: pad, display:pad, F.Cu at (154.9, 137.2)
- added REF**: pad, display:pad, F.Cu at (137.2, 119.4)
- added REF**: pad, display:pad, F.Cu at (144.8, 119.4)
- added REF**: pad, display:pad, F.Cu at (142.2, 116.8)
- added REF**: pad, display:pad, F.Cu at (144.8, 114.3)
- added REF**: pad, display:pad, F.Cu at (142.2, 111.8)
- added REF**: pad, display:pad, F.Cu at (139.7, 111.8)
- added REF**: pad, display:pad, F.Cu at (142.2, 119.4)
- added REF**: pad, display:pad, F.Cu at (139.7, 116.8)
- added REF**: pad, display:pad, F.Cu at (137.2, 116.8)
- added REF**: pad, display:pad, F.Cu at (144.8, 116.8)
- added REF**: pad, display:pad, F.Cu at (152.4, 137.2)
- added REF**: pad, display:pad, F.Cu at (139.7, 114.3)
- added REF**: pad, display:pad, F.Cu at (147.3, 137.2)
- added REF**: pad, display:pad, F.Cu at (149.9, 137.2)
- added REF**: pad, display:pad, F.Cu at (134.6, 137.2)
- added REF**: pad, display:pad, F.Cu at (165.1, 134.6)
- added REF**: pad, display:pad, F.Cu at (162.6, 134.6)
- added REF**: pad, display:pad, F.Cu at (160.0, 134.6)
- added REF**: pad, display:pad, F.Cu at (157.5, 134.6)
- added REF**: pad, display:pad, F.Cu at (155.0, 134.6)
- added REF**: pad, display:pad, F.Cu at (152.4, 134.6)
- added REF**: pad, display:pad, F.Cu at (149.9, 134.6)
- added REF**: pad, display:pad, F.Cu at (165.1, 132.1)
- added REF**: pad, display:pad, F.Cu at (154.9, 132.1)
- added REF**: pad, display:pad, F.Cu at (160.0, 132.1)
- added REF**: pad, display:pad, F.Cu at (137.2, 137.2)
- added REF**: pad, display:pad, F.Cu at (157.5, 132.1)
- added REF**: pad, display:pad, F.Cu at (162.6, 132.1)
- added REF**: pad, display:pad, F.Cu at (152.4, 132.1)
- added REF**: pad, display:pad, F.Cu at (165.1, 144.8)
- added REF**: pad, display:pad, F.Cu at (162.6, 142.2)
- added REF**: pad, display:pad, F.Cu at (165.1, 147.3)
- added REF**: pad, display:pad, F.Cu at (160.0, 144.8)
- added REF**: pad, display:pad, F.Cu at (160.0, 147.3)
- added REF**: pad, display:pad, F.Cu at (162.6, 147.3)
- added REF**: pad, display:pad, F.Cu at (160.0, 139.7)
- added REF**: pad, display:pad, F.Cu at (139.7, 137.2)
- added REF**: pad, display:pad, F.Cu at (157.5, 147.3)
- added REF**: pad, display:pad, F.Cu at (160.0, 142.2)
- added REF**: pad, display:pad, F.Cu at (165.1, 142.2)
- added REF**: pad, display:pad, F.Cu at (162.6, 139.7)
- added REF**: pad, display:pad, F.Cu at (157.5, 139.7)
- added REF**: pad, display:pad, F.Cu at (157.5, 142.2)
- added REF**: pad, display:pad, F.Cu at (165.1, 139.7)
- added REF**: pad, display:pad, F.Cu at (162.6, 144.8)
- added REF**: pad, display:pad, F.Cu at (157.5, 144.8)
- added REF**: pad, display:pad, F.Cu at (167.6, 132.1)
- added REF**: pad, display:pad, F.Cu at (142.2, 137.2)
- added REF**: pad, display:pad, F.Cu at (124.5, 124.5)
- added REF**: pad, display:pad, F.Cu at (119.4, 129.5)
- added REF**: pad, display:pad, F.Cu at (121.9, 127.0)
- added REF**: pad, display:pad, F.Cu at (124.5, 127.0)
- added REF**: pad, display:pad, F.Cu at (121.9, 129.5)
- added REF**: pad, display:pad, F.Cu at (124.5, 129.5)
- added REF**: pad, display:pad, F.Cu at (167.6, 129.5)
- added REF**: pad, display:pad, F.Cu at (170.2, 129.5)
- added REF**: pad, display:pad, F.Cu at (162.6, 129.5)
- added REF**: pad, display:pad, F.Cu at (165.1, 129.5)
- added REF**: pad, display:pad, F.Cu at (144.8, 134.6)
- added REF**: pad, display:pad, F.Cu at (157.5, 129.5)
- added REF**: pad, display:pad, F.Cu at (160.0, 129.5)
- added REF**: pad, display:pad, F.Cu at (142.2, 132.1)
- added REF**: pad, display:pad, F.Cu at (147.3, 132.1)
- added REF**: pad, display:pad, F.Cu at (144.8, 132.1)
- added REF**: pad, display:pad, F.Cu at (139.7, 132.1)
- added REF**: pad, display:pad, F.Cu at (129.5, 132.1)
- added REF**: pad, display:pad, F.Cu at (137.2, 132.1)
- added REF**: pad, display:pad, F.Cu at (134.6, 132.1)
- added REF**: pad, display:pad, F.Cu at (119.4, 132.1)
- added REF**: pad, display:pad, F.Cu at (142.2, 134.6)
- added REF**: pad, display:pad, F.Cu at (127.0, 132.1)
- added REF**: pad, display:pad, F.Cu at (124.5, 132.1)
- added REF**: pad, display:pad, F.Cu at (132.1, 132.1)
- added REF**: pad, display:pad, F.Cu at (121.9, 132.1)
- added REF**: pad, display:pad, F.Cu at (116.8, 132.1)
- added REF**: pad, display:pad, F.Cu at (147.3, 142.2)
- added REF**: pad, display:pad, F.Cu at (149.9, 147.3)
- added REF**: pad, display:pad, F.Cu at (152.4, 142.2)
- added REF**: pad, display:pad, F.Cu at (154.9, 139.7)
- added REF**: pad, display:pad, F.Cu at (147.3, 139.7)
- added REF**: pad, display:pad, F.Cu at (139.7, 134.6)
- added REF**: pad, display:pad, F.Cu at (147.3, 147.3)
- added REF**: pad, display:pad, F.Cu at (154.9, 147.3)
- added REF**: pad, display:pad, F.Cu at (152.4, 144.8)
- added REF**: pad, display:pad, F.Cu at (154.9, 142.2)
- added REF**: pad, display:pad, F.Cu at (152.4, 139.7)
- added REF**: pad, display:pad, F.Cu at (149.9, 139.7)
- added REF**: pad, display:pad, F.Cu at (152.4, 147.3)
- added REF**: pad, display:pad, F.Cu at (149.9, 144.8)
- added REF**: pad, display:pad, F.Cu at (147.3, 144.8)
- added REF**: pad, display:pad, F.Cu at (154.9, 144.8)
- added REF**: pad, display:pad, F.Cu at (137.2, 134.6)
- added REF**: pad, display:pad, F.Cu at (149.9, 142.2)
- added REF**: pad, display:pad, F.Cu at (147.3, 124.5)
- added REF**: pad, display:pad, F.Cu at (149.9, 129.5)
- added REF**: pad, display:pad, F.Cu at (152.4, 124.5)
- added REF**: pad, display:pad, F.Cu at (147.3, 121.9)
- added REF**: pad, display:pad, F.Cu at (147.3, 129.5)
- added REF**: pad, display:pad, F.Cu at (154.9, 129.5)
- added REF**: pad, display:pad, F.Cu at (152.4, 127.0)
- added REF**: pad, display:pad, F.Cu at (152.4, 121.9)
- added REF**: pad, display:pad, F.Cu at (149.9, 121.9)
- added TFT**: SPI_TFT, display:SPI_TFT, F.Cu at (140.8, 107.8)
Routing:
- net Net-(D7-Pad2): track 79.7 -> 76.7 mm
- net Net-(C1-Pad1): track 167.4 -> 170.3 mm
- net Net-(IC1-Pad31): track 123.2 -> 120.7 mm
- net (no net): vias 0 -> 3
Other:
- outline, holes or cut-outs redrawn
- board text added: "5V"
- board text added: "GND"
