File: regulator board/regulator board.sch (KiCad schematic (older format))
At the start: 101 parts, among them J1 Phoenix connector 01x04, J10 Screw terminal 01x02, J2 C14 socket https://bit.ly/2kj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, J3 Pin socket, J4 Phoenix connector 01x04, J5 Phoenix connector 01x04, J6 Screw terminal 01x02, J7 Phoenix connector 01x04, J8 Screw terminal 01x02, Q1 BSS84, Q2 BSS84, SW1 SW_Push_Dual, SW2 SW_Push_Dual, SW3 SW_Push_Dual, SW4 SW_Push_Dual, SW5 SW_Push_Dual, SW6 SW_Push_Dual, U1 MOC3063M, U10 MOC3063M, U11 PCF8574P https://bit.ly/2mbAL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, U12 PCF8574P https://bit.ly/2mbAL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, U13 DS2482S-100, U14 DS2482S-100, U2 PCF8574P https://bit.ly/2mbAL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, U3 MOC3063M, U4 MOC3063M, U5 MOC3063M, U6 MOC3063M, U7 ESP-32S https://bit.ly/2kIsByf, U8 MOC3063M, U9 MOC3063M

Commit message: Update PCB
Parts:
- removed J10, J6: Screw terminal 01x02, symbol Connector:Screw_Terminal_01x02
- removed J8: Screw terminal 01x02, TerminalBlock_Phoenix:TerminalBlock_Phoenix_MKDS-1,5-2_1x02_P5.00mm_Horizontal, symbol Connector:Screw_Terminal_01x02
- removed J?: Screw_Terminal_01x16, symbol Connector:Screw_Terminal_01x16
- removed U?: AMS1117-3.3 https://bit.ly/2kCiY4j, Converter_DCDC:Converter_DCDC_RECOM_R-78B-2.0_THT, symbol Regulator_Switching:R-78B5.0-2.0
- added J10, J7, J9: Conn_01x02_Female, Connector_PinSocket_2.54mm:PinSocket_1x02_P2.54mm_Vertical, symbol Connector:Conn_01x02_Female
- added J8: Conn_01x16_Female, Connector_PinSocket_2.54mm:PinSocket_1x16_P2.54mm_Vertical, symbol Connector:Conn_01x16_Female
- added U2: LM1117SX-3.3, Package_TO_SOT_SMD:TO-263-3_TabPin2, symbol Regulator_Linear:LM1117-3.3
- R14, R15: renamed from R?; footprint (none) -> Resistor_THT:R_Axial_DIN0204_L3.6mm_D1.6mm_P5.08mm_Horizontal
- R23: renamed from R29; footprint (none) -> Resistor_THT:R_Axial_DIN0204_L3.6mm_D1.6mm_P5.08mm_Horizontal
- R30: footprint (none) -> Resistor_THT:R_Axial_DIN0204_L3.6mm_D1.6mm_P5.08mm_Horizontal
- gave numbers to parts that had none: 4
- renumbered D14 to D10, D13 to D11, D11 to D13, D10 to D14, D9 to D15, D15 to D9, J2 to J1, J1 to J2, J7 to J6, Q1 to Q2, Q2 to Q3, R14 to R16, R15 to R17, R16 to R18, R17 to R19, R18 to R20, R19 to R21, R20 to R22, R21 to R24, R22 to R25, R24 to R26, R26 to R27, R23 to R29, R25 to R31, R27 to R32, R28 to R33, U9 to U10, U10 to U11, U11 to U12, U12 to U13, U13 to U14, U14 to U15, U2 to U3, U3 to U4, U4 to U5, U5 to U6, U6 to U7, U7 to U8, U8 to U9
Connections:
- net +3V3: now also U2.2 (VO); no longer C4.1
- net +5V: now also C4.1, J7.1 (Pin_1), J9.1 (Pin_1), U2.3 (VI)
- net GND: now also J7.2 (Pin_2), J9.2 (Pin_2), U2.1 (GND)
- net R1: now also J8.1 (Pin_1)
- net R10: now also J8.10 (Pin_10)
- net R11: now also J8.11 (Pin_11)
- net R12: now also J8.12 (Pin_12)
- net R13: now also J8.13 (Pin_13)
- net R14: now also J8.14 (Pin_14)
- net R15: now also J8.15 (Pin_15)
- net R16: now also J8.16 (Pin_16)
- net R2: now also J8.2 (Pin_2)
- net R3: now also J8.3 (Pin_3)
- net R4: now also J8.4 (Pin_4)
- net R5: now also J8.5 (Pin_5)
- net R6: now also J8.6 (Pin_6)
- net R7: now also J8.7 (Pin_7)
- net R8: now also J8.8 (Pin_8)
- net R9: now also J8.9 (Pin_9)
- net at Q2.2 (S), U14.2 (IO): now also J10.1 (Pin_1)
- net at Q3.2 (S), U15.2 (IO): now also J10.2 (Pin_2)
Other:
- moved on the sheet: C4

Commit message: Fix
Parts:
- removed C1, C2, C3, C4, C5, C6: 100nF, Capacitor_THT:C_Rect_L7.0mm_W2.0mm_P5.00mm, symbol Device:C
- removed C10, C11, C12, C13, C14, C7, C8, C9: 0.01uF, Capacitor_THT:C_Rect_L18.0mm_W5.0mm_P15.00mm_FKS3_FKP3, symbol Device:C
- removed D1, D10, D11, D12, D13, D14, D15, D16, D2, D3, D4, D5, D6, D7, D8, D9: LED, LED_THT:LED_D5.0mm, symbol Device:LED
- removed J1: C14 socket https://bit.ly/2kjjjZt, Connector_Wire:SolderWirePad_1x03_P5.715mm_Drill2mm, symbol Connector:Conn_WallSocket_Earth
- removed J10, J7, J9: Conn_01x02_Female, Connector_PinSocket_2.54mm:PinSocket_1x02_P2.54mm_Vertical, symbol Connector:Conn_01x02_Female
- removed J2, J4, J5, J6: Phoenix connector 01x04, Connector_Phoenix_MSTB:PhoenixContact_MSTBVA_2,5_4-G_1x04_P5.00mm_Vertical, symbol Connector:Conn_01x04_Female
- removed J3: Pin socket, Connector_PinSocket_2.54mm:PinSocket_1x04_P2.54mm_Vertical, symbol Connector:Conn_01x04_Female
- removed J8: Conn_01x16_Female, Connector_PinSocket_2.54mm:PinSocket_1x16_P2.54mm_Vertical, symbol Connector:Conn_01x16_Female
- removed PS1: Power supply https://bit.ly/2kBfKOu, Converter_ACDC:Converter_ACDC_HiLink_HLK-PMxx, symbol Converter_ACDC:HLK-PM03
- removed Q1, Q2, Q3: BSS84, Package_TO_SOT_SMD:SOT-23, symbol Transistor_FET:BSS84
- removed R1, R10, R12, R16, R18, R3, R5, R8: 330, Resistor_THT:R_Axial_DIN0204_L3.6mm_D1.6mm_P5.08mm_Horizontal, symbol Device:R
- removed R11, R13, R17, R19, R2, R4, R7, R9: 39, Resistor_THT:R_Axial_DIN0204_L3.6mm_D1.6mm_P5.08mm_Horizontal, symbol Device:R
- removed R14, R15: 4k7, Resistor_THT:R_Axial_DIN0204_L3.6mm_D1.6mm_P5.08mm_Horizontal, symbol Device:R
- removed R20, R21, R22, R24, R25, R26, R27, R28: 180, Resistor_THT:R_Axial_DIN0204_L3.6mm_D1.6mm_P5.08mm_Horizontal, symbol Device:R
- removed R23, R30: 100, Resistor_THT:R_Axial_DIN0204_L3.6mm_D1.6mm_P5.08mm_Horizontal, symbol Device:R
- removed R29, R31, R32, R33, R6: 10K, Resistor_THT:R_Axial_DIN0204_L3.6mm_D1.6mm_P5.08mm_Horizontal, symbol Device:R
- removed RV1: Varistor, Varistor:RV_Disc_D12mm_W3.9mm_P7.5mm, symbol Device:Varistor
- removed SW1, SW2: SW_Push_Dual, Button_Switch_THT:SW_TH_Tactile_Omron_B3F-10xx, symbol Switch:SW_Push_Dual
- removed SW3, SW4, SW5, SW6: SW_Push_Dual, Button_Switch_THT:Push_E-Switch_KS01Q01, symbol Switch:SW_Push_Dual
- removed TFT1: SPI TFT https://bit.ly/2lMnf5f, regulator board:SPI_TFT, symbol display:SPI_TFT
- removed U1, U10, U11, U4, U5, U6, U7, U9: MOC3063M, Package_DIP:DIP-6_W7.62mm_Socket, symbol Relay_SolidState:MOC3063M
- removed U12, U13, U16, U3: PCF8574P https://bit.ly/2mbALiV, Package_DIP:DIP-16_W7.62mm, symbol Interface_Expansion:PCF8574
- removed U14, U15: DS2482S-100, Package_SO:SOP-8_3.76x4.96mm_P1.27mm, symbol display:DS2482S-100
- removed U2: LM1117SX-3.3, Package_TO_SOT_SMD:TO-263-3_TabPin2, symbol Regulator_Linear:LM1117-3.3
- removed U8: ESP-32S https://bit.ly/2kIsByf, RF_Module:ESP32-WROOM-32, symbol RF_Module:ESP32-WROOM-32
Connections:
- no-connect marks 27 -> 0
Other:
- note removed: "AC 220V-DC 5V"
- note removed: "Boot"
- note removed: "Display"
- note removed: "Enable"
- note removed: "Ground\nFloor"
- note removed: "Keyboard"
- note removed: "Left\nNeutral\nRight\nEarth"
- note removed: "Power supply"
- note removed: "Pump switch"
- note removed: "Serial I/O"
- note removed: "Status indicators"
- note removed: "Tempature sensor controler"
